File: pump-monitor-interface-board/current_sense.sch (KiCad schematic (older format))
At the start: 33 parts, among them U1 TLV4333, U2 LMV331, U3 LMV321

Commit message: Design checklists
Parts:
- added C7: 0.1U, Capacitor_SMD:C_0805_2012Metric_Pad1.18x1.45mm_HandSolder, symbol pump-monitor-interface-board:C_0805
- added TP5: GND, TestPoint:TestPoint_Keystone_5000-5004_Miniature, symbol pump-monitor-interface-board:TestPoint
Connections:
- net +5V: now also C7.1
- net GND: now also C7.2, TP5.1
Changed lines of the file:
@@
 	1275 7400 1275 5500
 Wire Notes Line
-	1275 5500 3825 5500
-Wire Notes Line
-	3825 5500 3825 7400
-Wire Notes Line
-	3825 7400 1275 7400
+	4100 5500 4100 7400
 Wire Wire Line
 	1675 3425 2150 3425
@@
 Wire Wire Line
 	9575 3500 10050 3500
+$Comp
+L pump-monitor-interface-board:TestPoint TP5
+U 1 1 5F9D5811
+P 6150 6450
+F 0 "TP5" H 5950 6575 50  0000 L CNN
+F 1 "GND" H 5925 6500 50  0000 L CNN
+F 2 "TestPoint:TestPoint_Keystone_5000-5004_Miniature" H 6350 6450 50  0001 C CNN
+F 3 "~" H 6350 6450 50  0001 C CNN
+F 4 "n/a" H 6150 6450 50  0001 C CNN "In stock"
+F 5 "n/a" H 6150 6450 50  0001 C CNN "MPN"
+	1    6150 6450
+	1    0    0    -1
+$EndComp
+$Comp
+L power:GND #PWR?
+U 1 1 5F9D5C96
+P 6150 6450
+AR Path="/5F9D5C96" Ref="#PWR?"  Part="1"
+AR Path="/5F859606/5F9D5C96" Ref="#PWR0101"  Part="1"
+AR Path="/5F8A60BA/5F9D5C96" Ref="#PWR?"  Part="1"
+F 0 "#PWR0101" H 6150 6200 50  0001 C CNN
+F 1 "GND" H 6155 6277 50  0000 C CNN
+F 2 "" H 6150 6450 50  0001 C CNN
+F 3 "" H 6150 6450 50  0001 C CNN
+	1    6150 6450
+	1    0    0    -1
+$EndComp
+$Comp
+L power:+5V #PWR035
+U 1 1 5F9DE7D8
+P 3775 6650
+AR Path="/5F859606/5F9DE7D8" Ref="#PWR035"  Part="1"
+AR Path="/5F8A60BA/5F9DE7D8" Ref="#PWR?"  Part="1"
+F 0 "#PWR035" H 3775 6500 50  0001 C CNN
+F 1 "+5V" H 3790 6823 50  0000 C CNN
+F 2 "" H 3775 6650 50  0001 C CNN
+F 3 "" H 3775 6650 50  0001 C CNN
+	1    3775 6650
+	1    0    0    -1
+$EndComp
+$Comp
+L pump-monitor-interface-board:C_0805 C7
+U 1 1 5F9DE7E0
+P 3775 6800
+F 0 "C7" H 3890 6846 50  0000 L CNN
+F 1 "0.1U" H 3890 6755 50  0000 L CNN
+F 2 "Capacitor_SMD:C_0805_2012Metric_Pad1.18x1.45mm_HandSolder" H 3813 6650 50  0001 C CNN
+F 3 "" H 3775 6800 50  0001 C CNN
+F 4 "Y" H 3775 6800 50  0001 C CNN "In stock"
+F 5 "885012207098" H 3775 6800 50  0001 C CNN "MPN"
+	1    3775 6800
+	1    0    0    -1
+$EndComp
+$Comp
+L power:GND #PWR036
+U 1 1 5F9DE7E6
+P 3775 6950
+AR Path="/5F859606/5F9DE7E6" Ref="#PWR036"  Part="1"
+AR Path="/5F8A60BA/5F9DE7E6" Ref="#PWR?"  Part="1"
+F 0 "#PWR036" H 3775 6700 50  0001 C CNN
+F 1 "GND" H 3780 6777 50  0000 C CNN
+F 2 "" H 3775 6950 50  0001 C CNN
+F 3 "" H 3775 6950 50  0001 C CNN
+	1    3775 6950
+	1    0    0    -1
+$EndComp
+Wire Notes Line
+	1275 7400 4100 7400
+Wire Notes Line
+	1275 5500 4100 5500
 $EndSCHEMATC
