File: pump-monitor-interface-board/pump-monitor-interface-board.kicad_pcb (KiCad board)
At the start: 2 copper layers, 65 x 56.5 mm, 46 parts, among them J1 Conn_01x04, J2 RPI_HAT, J3 Conn_01x04, J4 Conn_01x02, J5 Conn_01x03, Q1 2N7002, U1 TLV4333, U2 LMV331, U3 LMV321

Commit message: Design checklists
Parts:
- added C7: 0.1U, Capacitor_SMD:C_0805_2012Metric_Pad1.18x1.45mm_HandSolder, F.Cu at (138.4, 129.7)
- added TP5: GND, TestPoint:TestPoint_Keystone_5000-5004_Miniature, F.Cu at (163.8, 106.2)
- moved R21 5.94 mm to (129.2, 132.3)
- moved R20 5.80 mm to (132.5, 131.5), turned to 270 degrees
- moved C5 4.92 mm to (131.4, 134.8)
- moved H1 0.50 mm to (113.5, 89.0)
- moved H3 0.50 mm to (171.5, 89.0)
- moved J2 0.50 mm to (118.4, 87.7)
Connections:
- U3 pad 1: Net-(C5-Pad1) -> +2V5
- U3 pad 3: +2V5 -> Net-(C5-Pad1)
Routing:
- net GND: track 23.8 -> 28.5 mm, vias 12 -> 17
- net +5V: track 17.0 -> 19.0 mm
- net +2V5: track 68.8 -> 70.2 mm
- net Net-(C5-Pad1): track 9.18 -> 8.01 mm
- net +3V3: track 60.7 -> 61.4 mm

Commit message: Tidying
Parts:
- J2: moved to B.Cu
- moved J3 18.5 mm to (115.0, 104.0)
- moved J1 16.0 mm to (115.0, 122.0)
- moved R1 16.0 mm to (118.3, 114.5)
- moved R2 16.0 mm to (117.4, 111.0)
- moved J2 2.59 mm to (118.4, 90.3), turned to 270 degrees
- moved R3 2.55 mm to (123.5, 127.0)
- moved R13 1.60 mm to (159.8, 100.3)
- moved R17 1.60 mm to (159.8, 96.0)
- moved TP4 1.60 mm to (163.5, 101.3)
Connections:
- J2 pad 10: ULTRASONIC_TRIGGER -> Net-(J2-Pad10)
- J2 pad 11: Net-(J2-Pad11) -> ULTRASONIC_ECHO
- J2 pad 12: TEMP_HUMIDITY -> Net-(J2-Pad12)
- J2 pad 13: Net-(J2-Pad13) -> ULTRASONIC_TRIGGER
- J2 pad 15: Net-(J2-Pad15) -> SSR
- J2 pad 16: SSR -> Net-(J2-Pad16)
- J2 pad 3: Net-(J2-Pad3) -> I2C_SDA
- J2 pad 37: Net-(J2-Pad37) -> CURRENT_SENSE
- J2 pad 40: CURRENT_SENSE -> Net-(J2-Pad40)
- J2 pad 5: Net-(J2-Pad5) -> I2C_SCL
- J2 pad 8: ULTRASONIC_ECHO -> Net-(J2-Pad8)
- J3 pad 2: TEMP_HUMIDITY -> I2C_SDA
- J3 pad 4: Net-(J3-Pad4) -> I2C_SCL
Routing:
- net TEMP_HUMIDITY: track 38.5 -> 0.00 mm, vias 1 -> 0
- net +3V3: track 61.4 -> 40.2 mm
- net I2C_SDA: track 0.00 -> 18.1 mm
- net ULTRASONIC_TRIGGER: track 21.4 -> 38.1 mm
- net ULTRASONIC_ECHO: track 13.0 -> 28.5 mm
- net +5V: track 19.0 -> 7.57 mm, vias 4 -> 0
- net I2C_SCL: track 0.00 -> 11.0 mm
- net GND: track 28.5 -> 20.3 mm, vias 17 -> 18
- net Net-(Q1-Pad1): track 3.02 -> 4.56 mm
- net SSR: track 42.6 -> 41.6 mm, vias 1 -> 2
- net Net-(R13-Pad2): track 12.0 -> 11.3 mm
- net CURRENT_SENSE: track 11.2 -> 11.9 mm
Other:
- board text added: "SCL"
- board text added: "SDA"
- board text removed: "DATA"
- board text removed: "NC"
