File: pump-monitor-interface-board/pump-monitor-interface-board.sch (KiCad schematic (older format))
At the start: 13 parts, among them J1 Conn_01x04, J2 RPI_HAT, J3 Conn_01x04, J4 Conn_01x02, J5 Conn_01x03, Q1 2N7002

Commit message: Tidying
Connections:
- net CURRENT_SENSE: now also J2.37 (GPIO26); no longer J2.40 (GPIO21)
- net SSR: now also J2.15 (GPIO22); no longer J2.16 (GPIO23)
- net ULTRASONIC_ECHO: now also J2.11 (GPIO17); no longer J2.8 (GPIO14)
- net ULTRASONIC_TRIGGER: now also J2.13 (GPIO27); no longer J2.10 (GPIO15)
- net I2C_SDA: now reaches J2.3 (GPIO2)
- net I2C_SDA: now also J3.2 (Pin_2)
- net I2C_SCL: now reaches J2.5 (GPIO3)
- net I2C_SCL: now also J3.4 (Pin_4)
- net TEMP_HUMIDITY: no longer names the net of J2.12 (GPIO18)
- net TEMP_HUMIDITY: no longer J3.2 (Pin_2)
- no-connect marks 24 -> 23
Other:
- note added: "Connect to Adafruit\n3721 temperature\nand humidity sensor."
- note added: "SCL"
- note removed: "Connect to Seeed\nAM2311A temperature\nand humidity sensor."
- note removed: "NC"
- moved on the sheet: J2
